File: STEP100-200-switch-id-shield/STEP100-200-switch-id-shield.kicad_pcb (KiCad board)
At the start: 2 copper layers, 50 x 51 mm, 13 parts, among them J1 Conn_01x08, J2 Conn_01x08, J3 Conn_01x06, J4 Conn_01x10, J5 Conn_01x03, J6 Conn_02x04_Odd_Even, J7 Conn_01x03, J8 Conn_01x03, J9 Conn_01x03, SW1 SW_DIP_x04

Commit message: version 2 PCBs
Connections:
- net Net-(A1-D6) renamed /DIP_2
- net Net-(A1-D7) renamed /DIP_3
- A1 pad 12: Net-(A1-A3) -> /LIMIT_1
- A1 pad 20: Net-(A1-D5) -> /DIP_4
- A1 pad 9: /LIMIT_1 -> /DIP_1
- J1 pad 3: Net-(A1-D5) -> /DIP_4
- J3 pad 1: /LIMIT_1 -> /DIP_1
- J3 pad 4: Net-(A1-A3) -> /LIMIT_1
- SW1 pad 1: Net-(A1-D5) -> /DIP_1
- SW1 pad 4: Net-(A1-D9) -> /DIP_4
Routing:
- net /DIP_1: track 0.00 -> 63.3 mm
- net Net-(A1-D9): track 25.9 -> 2.54 mm
- net /DIP_4: track 0.00 -> 20.6 mm
- net Net-(A1-D5): track 11.0 -> 0.00 mm
- net /LIMIT_1: track 55.7 -> 59.9 mm, vias 0 -> 1
- net Net-(A1-A3): track 2.54 -> 0.00 mm
- net /DIP_2: track 14.6 -> 15.3 mm
- net GND: vias 0 -> 2
Other:
- board text added: "A3"
- board text added: "D5"
- board text added: "D6"
- board text added: "D7"
- board text added: "rev 2.0 / 2024-12-10"
- board text removed: "Sensors + ID switch shield"
- board text removed: "rev 1.0 / 2024-03-26"
