File: STEP100-200-switch-id-shield/STEP100-200-switch-id-shield.kicad_sch (KiCad schematic)
At the start: 12 parts, among them J1 Conn_01x08, J2 Conn_01x08, J3 Conn_01x06, J4 Conn_01x10, J5 Conn_01x03, J6 Conn_02x04_Odd_Even, J7 Conn_01x03, J8 Conn_01x03, J9 Conn_01x03, SW1 SW_DIP_x04

Commit message: version 2 PCBs
Connections:
- net LIMIT_1: now also A1.12 (A3), J3.4 (Pin_4); no longer A1.9 (A0), J3.1 (Pin_1)
- net at A1.24 (D9), J4.9 (Pin_9): no longer SW1.4
- net DIP_4: now reaches A1.20 (D5), J1.3 (Pin_3)
- net DIP_4: now also SW1.4; no longer SW1.1
- net DIP_2: now reaches A1.21 (D6), J1.2 (Pin_2), SW1.2
- net DIP_3: now reaches A1.22 (D7), J1.1 (Pin_1), SW1.3
- new net DIP_1: A1.9 (A0), J3.1 (Pin_1), SW1.1
Other:
- company: (none) -> Ponoor Experiments inc.
- title: (none) -> Switch ID shield for STEP100 and STEP200
- moved on the sheet: JP1, SW1
