File: STEP200-XA-motor-connector/STEP200-XA-motor-connector.kicad_pcb (KiCad board)
At the start: 2 copper layers, 58 x 21 mm, 6 parts, among them J1 Conn_01x04_Pin, J2 Conn_01x04_Socket, J3 Conn_01x04_Pin, J4 Conn_01x04_Socket, J5 Conn_01x02_Pin, J6 Conn_01x02_Socket

Commit message: version 2 PCBs
Parts:
- moved J1 1.00 mm to (95.0, 76.0)
- moved J2 1.00 mm to (97.2, 64.0)
- moved J3 1.00 mm to (133.0, 76.0)
- moved J4 1.00 mm to (135.2, 64.0)
Other:
- board size 58 x 21 mm -> 56 x 21 mm
- board text added: "Ponoor Experiments rev.2024-12-10"
- board text removed: "Ponoor Experiments rev.2024-04-18"
